File: include/digital-in.kicad_sch (KiCad schematic)
At the start: 5 parts, among them U9 EL817

Commit message: slave-8in-8out-0.2
Parts:
- R3: renamed from R44; LCSC C25917 -> C25130
- R4: renamed from R45; LCSC C25917 -> C25130
- renumbered D23 to D9, R46 to R5, U9 to U2
Changed lines of the file:
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@@
   (symbol (lib_id "Device:R") (at 71.12 48.26 270)
     (in_bom yes) (on_board yes)
-    (property "Reference" "R44" (id 0) (at 71.12 43.0022 90))
+    (property "Reference" "R3" (id 0) (at 71.12 43.0022 90))
     (property "Value" "680" (id 1) (at 71.12 45.3136 90))
     (property "Footprint" "Resistor_SMD:R_0402_1005Metric" (id 2) (at 71.12 46.482 90)
@@
       (effects (font (size 1.27 1.27)) hide)
     )
-    (property "LCSC" "C25917" (id 4) (at 71.12 48.26 90)
+    (property "LCSC" "C25130" (id 4) (at 71.12 48.26 90)
       (effects (font (size 1.27 1.27)) hide)
     )
@@
   (symbol (lib_id "Device:R") (at 78.74 36.83 270)
     (in_bom yes) (on_board yes)
-    (property "Reference" "R45" (id 0) (at 78.74 31.5722 90))
+    (property "Reference" "R4" (id 0) (at 78.74 31.5722 90))
     (property "Value" "680" (id 1) (at 78.74 33.8836 90))
     (property "Footprint" "Resistor_SMD:R_0402_1005Metric" (id 2) (at 78.74 35.052 90)
@@
       (effects (font (size 1.27 1.27)) hide)
     )
-    (property "LCSC" "C25917" (id 4) (at 78.74 36.83 90)
+    (property "LCSC" "C25130" (id 4) (at 78.74 36.83 90)
       (effects (font (size 1.27 1.27)) hide)
     )
@@
   (symbol (lib_id "Device:R") (at 97.79 45.72 180)
     (in_bom yes) (on_board yes)
-    (property "Reference" "R46" (id 0) (at 103.0478 45.72 90))
+    (property "Reference" "R5" (id 0) (at 103.0478 45.72 90))
     (property "Value" "10k" (id 1) (at 100.7364 45.72 90))
     (property "Footprint" "Resistor_SMD:R_0402_1005Metric" (id 2) (at 99.568 45.72 90)
@@
   (symbol (lib_id "Device:LED") (at 63.5 48.26 0)
     (in_bom yes) (on_board yes) (fields_autoplaced)
-    (property "Reference" "D23" (id 0) (at 63.3095 41.91 0))
+    (property "Reference" "D9" (id 0) (at 63.3095 41.91 0))
     (property "Value" "LED" (id 1) (at 63.3095 44.45 0))
     (property "Footprint" "LED_SMD:LED_0805_2012Metric" (id 2) (at 63.5 48.26 0)
@@
   (symbol (lib_id "jlcpcb:EL817") (at 90.17 39.37 0)
     (in_bom yes) (on_board yes)
-    (property "Reference" "U9" (id 0) (at 90.17 31.115 0))
+    (property "Reference" "U2" (id 0) (at 90.17 31.115 0))
     (property "Value" "EL817" (id 1) (at 90.17 33.4264 0))
     (property "Footprint" "jlcpcb:EL817" (id 2) (at 111.76 44.45 0)

Commit message: update slave-8in-8out labels
Parts:
- renumbered D9 to D23, R3 to R44, R4 to R45, R5 to R46, U2 to U9
Changed lines of the file:
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@@
   (symbol (lib_id "Device:R") (at 71.12 48.26 270)
     (in_bom yes) (on_board yes)
-    (property "Reference" "R3" (id 0) (at 71.12 43.0022 90))
+    (property "Reference" "R44" (id 0) (at 71.12 43.0022 90))
     (property "Value" "680" (id 1) (at 71.12 45.3136 90))
     (property "Footprint" "Resistor_SMD:R_0402_1005Metric" (id 2) (at 71.12 46.482 90)
@@
   (symbol (lib_id "Device:R") (at 78.74 36.83 270)
     (in_bom yes) (on_board yes)
-    (property "Reference" "R4" (id 0) (at 78.74 31.5722 90))
+    (property "Reference" "R45" (id 0) (at 78.74 31.5722 90))
     (property "Value" "680" (id 1) (at 78.74 33.8836 90))
     (property "Footprint" "Resistor_SMD:R_0402_1005Metric" (id 2) (at 78.74 35.052 90)
@@
   (symbol (lib_id "Device:R") (at 97.79 45.72 180)
     (in_bom yes) (on_board yes)
-    (property "Reference" "R5" (id 0) (at 103.0478 45.72 90))
+    (property "Reference" "R46" (id 0) (at 103.0478 45.72 90))
     (property "Value" "10k" (id 1) (at 100.7364 45.72 90))
     (property "Footprint" "Resistor_SMD:R_0402_1005Metric" (id 2) (at 99.568 45.72 90)
@@
   (symbol (lib_id "Device:LED") (at 63.5 48.26 0)
     (in_bom yes) (on_board yes) (fields_autoplaced)
-    (property "Reference" "D9" (id 0) (at 63.3095 41.91 0))
+    (property "Reference" "D23" (id 0) (at 63.3095 41.91 0))
     (property "Value" "LED" (id 1) (at 63.3095 44.45 0))
     (property "Footprint" "LED_SMD:LED_0805_2012Metric" (id 2) (at 63.5 48.26 0)
@@
   (symbol (lib_id "jlcpcb:EL817") (at 90.17 39.37 0)
     (in_bom yes) (on_board yes)
-    (property "Reference" "U2" (id 0) (at 90.17 31.115 0))
+    (property "Reference" "U9" (id 0) (at 90.17 31.115 0))
     (property "Value" "EL817" (id 1) (at 90.17 33.4264 0))
     (property "Footprint" "jlcpcb:EL817" (id 2) (at 111.76 44.45 0)
