File: slave-8in-8out/slave-8in-8out.kicad_sch (KiCad schematic)
At the start: 39 parts, among them J1 Conn_01x06_Male, J2 Screw_Terminal_01x02, J3 Conn_01x06_Female, J4 Screw_Terminal_01x04, J5 Screw_Terminal_01x04, J6 Screw_Terminal_01x04, J7 Screw_Terminal_01x04, J8 Conn_01x10_Male, J9 Screw_Terminal_01x02, SW1 SW_DIP_x05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

Commit message: add PCF8575 to slave-8in-8out
Parts:
- removed R11: 10k, Resistor_SMD:R_0402_1005Metric, symbol Device:R
- removed U1: MCP23017_SO, Package_SO:SOIC-28W_7.5x17.9mm_P1.27mm, symbol slave-8in-8out-rescue:MCP23017_SO-Interface_Expansion
- added U1: PCF8575, Package_SO:SSOP-24_5.3x8.2mm_P0.65mm, symbol custom:PCF8575
Connections:
- net +3V3: now also U1.24 (VCC)
- net A0: now also U1.21 (A0)
- net A1: now also U1.2 (A1)
- net A2: now also U1.3 (A2)
- net GND: now also U1.12 (GND)
- net GPA0: now also D8.2 (A), U1.13 (P10)
- net GPA1: now also D7.2 (A), U1.14 (P11); no longer D8.2 (A)
- net GPA2: now also U1.15 (P12)
- net GPA3: now also U1.16 (P13)
- net GPA4: now also U1.17 (P14)
- net GPA5: now also U1.18 (P15)
- net GPA6: now also U1.19 (P16)
- net GPA7: now also U1.20 (P17)
- net GPB0: now also U1.4 (P00)
- net GPB1: now also U1.5 (P01)
- net GPB2: now also U1.6 (P02)
- net GPB3: now also U1.7 (P03)
- net GPB4: now also U1.8 (P04)
- net GPB5: now also U1.9 (P05)
- net GPB6: now also U1.10 (P06)
- net GPB7: now also U1.11 (P07); no longer D7.2 (A)
- net SCL: now also U1.22 (SCL)
- net SDA: now also U1.23 (SDA)
- no-connect marks 0 -> 1
