File: new-slave/new-slave.kicad_sch (KiCad schematic)
At the start: 5 parts, among them J1 Conn_01x06_Male, J2 Conn_01x06_Male, J3 Conn_01x06_Female, J4 Screw_Terminal_01x03, U1 RS485-TTL-Board

Commit message: slave-modbus-1.0
Parts:
- removed J4: Screw_Terminal_01x03, TerminalBlock_Phoenix:TerminalBlock_Phoenix_PT-1,5-3-3.5-H_1x03_P3.50mm_Horizontal, symbol Connector:Screw_Terminal_01x03
- removed U1: RS485-TTL-Board, boards:RS485-TTL-Board-DsdTech, symbol boards:RS485-TTL-Board
- added H1, H2, H3, H4: MountingHole, MountingHole:MountingHole_3.2mm_M3, symbol Mechanical:MountingHole
- added J4: Conn_01x06_Female, Connector_PinSocket_2.54mm:PinSocket_1x06_P2.54mm_Horizontal, symbol Connector:Conn_01x06_Female
Connections:
- net GPIO14: now also J4.3 (Pin_3)
- net GPIO15: now also J4.4 (Pin_4)
- net GPIO35: now also J4.5 (Pin_5)
- net GPIO36: now also J4.6 (Pin_6)
- net GPIO4: now also J4.1 (Pin_1)
- net GPIO5: now also J4.2 (Pin_2)
- net +24V renamed +5V
